File: ligra_back/ligra_back.kicad_pcb (KiCad board)
At the start: 2 copper layers, 106.7 x 106.7 mm, 61 parts, among them J1 Mount, J10 USB-vertical_footprint, J11 USB_C_Receptacle_PowerOnly_6P, J2 Mount, J3 Mount, J4 Mount, J5 POWER, J6 POWER, J7 LED, J8 FAN, J9 Motor, Q1 BC807, Q2 AO3401A, Q3 BC807, SW2 Reverse, U1 MAX22202ATC+, U2 AL8843, U3 NCP1117-5_SOT223, U4 NCP1117-12_SOT223, U5 NCP1117-3.3_SOT223, U6 NE555

Commit message: updated back to v1.2.0
Parts:
- removed C18: 100n, otter:C_0603
- removed D3, D4: D210, Diode_SMD:D_SOD-123F
- removed JP2: jmp, otter:JMP_2_1
- removed R11: TBD, otter:R_0603
- removed U1: MAX22202ATC+, otter:TDFN12-3x3
- removed U3: NCP1117-5_SOT223, Package_TO_SOT_SMD:SOT-223-3_TabPin2
- removed U6: NE555, Package_SO:SOIC-8_3.9x4.9mm_P1.27mm
- added C19: 100n, otter:C_0603, B.Cu at (228.4, -97.1)
- added D5: LED, otter:LED_0603_1608Metric, B.Cu at (249.4, -94.0)
- added J12: XT60, Connector_AMASS:AMASS_XT60IPW-M_1x03_P7.20mm_Horizontal, B.Cu at (213.6, -63.0)
- added P1: TC2030-CTX-Tag-Connect, otter:TC2030, F.Cu at (249.4, -110.7)
- added R12: 5k1, otter:R_0603, B.Cu at (229.3, -98.0)
- added R13: 5k1, otter:R_0603, B.Cu at (249.0, -92.5)
- added U7: STM32F030F4Px, Package_SO:TSSOP-20_4.4x6.5mm_P0.65mm, B.Cu at (223.1, -99.5)
- added U8: DRV8231, Package_SO:SOIC-8-1EP_3.9x4.9mm_P1.27mm_EP2.62x3.51mm, B.Cu at (221.5, -88.9)
- C1, C3, C4: value 4u7 -> 100n; footprint otter:C_0805 -> otter:C_0603
- C17: value 1n -> 100n
- L2: footprint Inductor_SMD:L_Taiyo-Yuden_MD-5050 -> Inductor_SMD:L_Taiyo-Yuden_NR-80xx
- R1: value 5k1 -> R33; footprint otter:R_0603 -> otter:R_0805
- R10: value TBD -> LDR
- R2: value DNP -> 5k1
- R3: value 100 -> 5k1
- SW2: value Reverse -> SW_SP3T; footprint Button_Switch_THT:SW_CuK_JS202011CQN_DPDT_Straight -> otter:SW_3S
- moved C4 48.0 mm to (225.8, -94.5), turned to 135 degrees
- moved C2 44.1 mm to (211.0, -90.7), turned to 180 degrees
- moved JP1 42.9 mm to (207.8, -91.4), turned to 180 degrees
- moved R10 41.1 mm to (249.4, -115.2), turned to 180 degrees
- moved U4 36.6 mm to (208.8, -85.2), turned to 90 degrees
- moved C13 34.3 mm to (206.5, -94.2), turned to 0 degrees
- moved C14 34.1 mm to (209.8, -94.2), turned to 180 degrees
- moved C3 26.5 mm to (219.4, -103.3)
- moved C11 25.4 mm to (217.8, -92.2)
- moved U5 24.1 mm to (208.8, -99.5), turned to 90 degrees
- moved SW2 18.7 mm to (200.0, -140.0)
- moved C17 16.1 mm to (226.7, -95.4), turned to 135 degrees
- moved C15 12.8 mm to (213.7, -75.5), turned to 45 degrees
- moved C16 12.3 mm to (216.6, -100.8), turned to -45 degrees
- moved RV2 11.6 mm to (183.0, -134.8)
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Connections:
- C1 pad 2: Net-(U1-V18) -> +3V3
- C11 pad 2: Net-(U2-CTRL) -> Net-(U8-VREF)
- C12 pad 1: +5V -> +12V
- C15 pad 1: +5V -> +12V
- C16 pad 1: Net-(U6-CV) -> GND
- C16 pad 2: GND -> Net-(U7-PA5)
- C3 pad 2: +5V -> +3V3
- C4 pad 1: VBUS -> GND
- C4 pad 2: GND -> Net-(U7-PA1)
- C6 pad 2: +5V -> +12V
- R1 pad 1: GND -> Net-(U8-ISEN)
- R1 pad 2: Net-(U1-ILIM) -> GND
- R10 pad 1: +3V3 -> GND
- R10 pad 2: Net-(R10-Pad2) -> Net-(U7-PA5)
- R2 pad 1: GND -> Net-(U7-PA4)
- R2 pad 2: Net-(U1-ISEN) -> Net-(U8-VREF)
- R3 pad 1: +5V -> Net-(U7-PA5)
- R3 pad 2: Net-(D3-K) -> +3V3
- RV1 pad 1: Net-(R10-Pad2) -> GND
- RV1 pad 2: Net-(U2-CTRL) -> Net-(U7-PA1)
- RV1 pad 3: Net-(R11-Pad1) -> +3V3
- RV2 pad 1: Net-(D3-A) -> GND
- RV2 pad 3: Net-(D4-K) -> +3V3
- SW2 pad 1: GND -> Net-(U7-PA7)
- SW2 pad 3: +5V -> GND
- SW2 pad 4: (no net) -> unconnected-(SW2-Pad4)
- U2 pad 5: Net-(U2-CTRL) -> LED_CONTROL
Routing:
- net +3V3: track 20.0 -> 150.2 mm, vias 0 -> 5
- net +5V: track 120.1 -> 0.00 mm, vias 8 -> 0
- net Net-(U7-PA1): track 0.00 -> 66.7 mm, vias 0 -> 2
- net Net-(U7-PA7): track 0.00 -> 58.3 mm, vias 0 -> 4
- net Net-(D3-K): track 50.6 -> 0.00 mm, vias 2 -> 0
- net Net-(J8-Pin_2): track 3.28 -> 48.6 mm, vias 0 -> 3
- net Net-(U7-PA5): track 0.00 -> 44.3 mm, vias 0 -> 2
- net NRST: track 0.00 -> 35.4 mm, vias 0 -> 1
- net +12V: track 11.3 -> 44.7 mm
- net SWCLK: track 0.00 -> 30.0 mm, vias 0 -> 1
- net SWDIO: track 0.00 -> 29.5 mm, vias 0 -> 1
- net Net-(D5-A): track 0.00 -> 28.5 mm
- net LED_CONTROL: track 0.00 -> 27.4 mm, vias 0 -> 4
- net Net-(U2-CTRL): track 23.2 -> 0.00 mm, vias 2 -> 0
- net Net-(U7-PA2): track 0.00 -> 12.9 mm, vias 0 -> 2
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Other:
- board text added: "+ -"
- board text added: "- +"
- board text added: "A B"
- board text added: "FAN"
- board text added: "LDR"
- board text added: "LED"
- board text added: "MODE"
- board text added: "MOT"
- board text added: "MOTOR"
- board text added: "NC NC + GND"
