File: ligra_back/ligra_back.kicad_sch (KiCad schematic)
At the start: 59 parts, among them J1 Mount, J10 USB-vertical_footprint, J11 USB_C_Receptacle_PowerOnly_6P, J2 Mount, J3 Mount, J4 Mount, J5 POWER, J6 POWER, J7 LED, J8 FAN, J9 Motor, Q1 BC807, Q2 AO3401A, Q3 BC807, SW2 Reverse, U1 MAX22202ATC+, U2 AL8843, U3 NCP1117-5_SOT223, U4 NCP1117-12_SOT223, U5 NCP1117-3.3_SOT223, U6 NE555

Commit message: updated back to v1.2.0
Parts:
- removed C28 (x3): 100n, otter:C_0603, symbol Device:C_Small
- removed C28: 1n, otter:C_0603, symbol Device:C_Small
- removed C29 (x3): 4u7, otter:C_0805, symbol Device:C_Small
- removed D3, D4: D210, Diode_SMD:D_SOD-123F, symbol Device:D_Small
- removed JP2: jmp, otter:JMP_2_1, symbol Jumper:SolderJumper_3_Bridged12
- removed R10: DNP, otter:R_0603, symbol Device:R_Small
- removed R10 (x2): 5k1, otter:R_0603, symbol Device:R_Small
- removed R10: 2k2, otter:R_0603, symbol Device:R_Small
- removed R10: 100, otter:R_0603, symbol Device:R_Small
- removed SW2: Reverse, Button_Switch_THT:SW_CuK_JS202011CQN_DPDT_Straight, symbol Switch:SW_SPDT
- removed U1: MAX22202ATC+, otter:TDFN12-3x3, symbol otter:MAX22202ATC+
- removed U3: NCP1117-5_SOT223, Package_TO_SOT_SMD:SOT-223-3_TabPin2, symbol Regulator_Linear:NCP1117-3.3_SOT223
- removed U6: NE555, Package_SO:SOIC-8_3.9x4.9mm_P1.27mm, symbol otter:NE555
- added C1, C11, C16, C17, C19, C3, C4: 100n, otter:C_0603, symbol Device:C_Small
- added D5: LED, otter:LED_0603_1608Metric, symbol Device:LED
- added J12: XT60, Connector_AMASS:AMASS_XT60IPW-M_1x03_P7.20mm_Horizontal, symbol Connector_Generic:Conn_01x02
- added P1: TC2030-CTX-Tag-Connect, otter:TC2030, symbol otter:TC2030-CTX-Tag-Connect
- added R1: R33, otter:R_0805, symbol Device:R_Small
- added R10: LDR, otter:R_0603, symbol Device:R_Small
- added R12, R13, R2, R3: 5k1, otter:R_0603, symbol Device:R_Small
- added SW2: SW_SP3T, otter:SW_3S, symbol Switch:SW_SP3T
- added U7: STM32F030F4Px, Package_SO:TSSOP-20_4.4x6.5mm_P0.65mm, symbol MCU_ST_STM32F0:STM32F030F4Px
- added U8: DRV8231, Package_SO:SOIC-8-1EP_3.9x4.9mm_P1.27mm_EP2.62x3.51mm, symbol otter:DRV8231
- L1: footprint Inductor_SMD:L_Taiyo-Yuden_MD-5050 -> Inductor_SMD:L_Taiyo-Yuden_NR-80xx
Connections:
- net +5V is gone; now on net +12V: C15.1, C28.1, C29.2
- net +12V: now also U8.5 (VM)
- net +3V3: now also RV1.3, RV2.3, C1.2, C3.2, P1.1 (VCC), R3.2, U7.16 (VDD), U7.5 (VDDA)
- net GND: now also RV1.1, RV2.1, C1.1, C11.1, C16.1, C17.1, C19.1, C3.1, C4.1, J12.1 (Pin_1), P1.5 (GND), R1.2, R10.1, R12.1, R13.1, SW2.3, U7.15 (VSS), U8.1 (GND), U8.9 (GND)
- net VBUS: now also J12.2 (Pin_2)
- net at RV2.2: now also C17.2, U7.6 (PA0)
- net at RV1.2: now also C4.2, U7.7 (PA1); no longer U2.5 (CTRL)
- net at J9.2 (Pin_2): now also U8.8 (OUT2)
- net at J9.1 (Pin_1): now also U8.6 (OUT1)
- new net: U7.8 (PA2), U8.2 (IN2)
- new net: U7.9 (PA3), U8.3 (IN1)
- new net: C11.2, R2.2, U8.4 (VREF)
- new net: R1.1, U8.7 (ISEN)
- new net: R2.1, U7.10 (PA4)
- new net: D5.1 (K), R13.2
- new net: C16.2, R10.2, R3.1, U7.11 (PA5)
- new net: R12.2, U7.1 (BOOT0)
- new net: SW2.1, U7.13 (PA7)
- new net: SW2.2, U7.17 (PA9)
- new net: D5.2 (A), U7.2 (PF0)
- new net LED_CONTROL: U2.5 (CTRL), U7.12 (PA6)
- new net NRST: C19.2, P1.3 (~{RESET}), U7.4 (NRST)
- new net SWCLK: P1.4 (SWCLK/TCK), U7.20 (PA14)
- new net SWDIO: P1.2 (SWDIO/TMS), U7.19 (PA13)
- no-connect marks 3 -> 6
Other:
- note removed: ">0.4V 10% <2.5V 100%"
- moved on the sheet: C15, C28, C29, C7, D1, D2, J5, J6, J7, L1, R9, U2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
